Commit message: chitu_amp 学出来是趴着的,怀疑数据集没有导入正确

File: resources/robots/chitu/urdf/chitu.urdf (robot description, URDF)
Before this commit: robot chitu_max, 22 links, 21 joints
Links:
- removed link FL_FOOT
- removed link FL_FT_wrist
- removed link FL_calf
- removed link FL_hip
- removed link FL_thigh
- removed link FR_FOOT
- removed link FR_FT_wrist
- removed link FR_calf
- removed link FR_hip
- removed link FR_thigh
- removed link RL_FOOT
- removed link RL_FT_wrist
- removed link RL_calf
- removed link RL_hip
- removed link RL_thigh
- removed link RR_FOOT
- removed link RR_FT_wrist
- removed link RR_calf
- removed link RR_hip
- removed link RR_thigh
- added link LF_FOOT, mass 0.1; collision sphere radius=0.041; visual sphere radius=0.041
- added link LF_FT_wrist, mass 0.0001; visual sphere radius=0.0001
- added link LF_calf, mass 0.71704; collision box size=0.124 0.03 0.03; collision box size=0.26 0.03 0.03
- added link LF_hip, mass 3.7016; collision cylinder length=0.24 radius=0.06; visual mesh filename=../meshes/LFpitch_Link.STL
- added link LF_thigh, mass 5.093; collision box size=0.04 0.23 0.04; visual mesh filename=../meshes/LFthigh_Link.STL
- added link LH_FOOT, mass 0.1; collision sphere radius=0.041; visual sphere radius=0.041
- added link LH_FT_wrist, mass 0.0001; visual sphere radius=0.0001
- added link LH_calf, mass 0.71704; collision box size=0.124 0.03 0.03; collision box size=0.26 0.03 0.03
- added link LH_hip, mass 3.7016; collision cylinder length=0.24 radius=0.06; visual mesh filename=../meshes/LBpitch_Link.STL
- added link LH_thigh, mass 5.093; collision box size=0.04 0.23 0.04; visual mesh filename=../meshes/LBthigh_Link.STL
- added link RF_FOOT, mass 0.1; collision sphere radius=0.041; visual sphere radius=0.041
- added link RF_FT_wrist, mass 0.0001; visual sphere radius=0.0001
- added link RF_calf, mass 0.71704; collision box size=0.124 0.03 0.03; collision box size=0.26 0.03 0.03
- added link RF_hip, mass 3.7016; collision cylinder length=0.24 radius=0.06; visual mesh filename=../meshes/RFpitch_Link.STL
- added link RF_thigh, mass 5.093; collision box size=0.04 0.23 0.04; visual mesh filename=../meshes/RFthigh_Link.STL
- added link RH_FOOT, mass 0.1; collision sphere radius=0.041; visual sphere radius=0.041
- added link RH_FT_wrist, mass 0.0001; visual sphere radius=0.0001
- added link RH_calf, mass 0.71704; collision box size=0.124 0.03 0.03; collision box size=0.26 0.03 0.03
- added link RH_hip, mass 3.7016; collision cylinder length=0.24 radius=0.06; visual mesh filename=../meshes/RBpitch_Link.STL
- added link RH_thigh, mass 5.093; collision box size=0.04 0.23 0.04; visual mesh filename=../meshes/RBthigh_Link.STL
Joints:
- removed joint FL_calf_joint
- removed joint FL_foot_fixed
- removed joint FL_ft_joint
- removed joint FL_hip_joint
- removed joint FL_thigh_joint
- removed joint FR_calf_joint
- removed joint FR_foot_fixed
- removed joint FR_ft_joint
- removed joint FR_hip_joint
- removed joint FR_thigh_joint
- removed joint RL_calf_joint
- removed joint RL_foot_fixed
- removed joint RL_ft_joint
- removed joint RL_hip_joint
- removed joint RL_thigh_joint
- removed joint RR_calf_joint
- removed joint RR_foot_fixed
- removed joint RR_ft_joint
- removed joint RR_hip_joint
- removed joint RR_thigh_joint
- added joint LF_HAA: type revolute, parent base, child LF_hip, origin xyz=0.301 0.10557 0 rpy=0 0 0, axis 1 0 0, limit lower=-0.7854 upper=0.7854 effort=299 velocity=9.14
- added joint LF_HFE: type revolute, parent LF_hip, child LF_thigh, origin xyz=0.0795 0.0272 0 rpy=0 0 0, axis 0 1 0, limit lower=-2.618 upper=2.618 effort=299 velocity=9.14
- added joint LF_KFE: type revolute, parent LF_thigh, child LF_calf, origin xyz=-0.24748 0.12015 -0.24752 rpy=0 0 0, axis 0 1 0, limit lower=-1.1345 upper=0.7854 effort=299 velocity=9.14
- added joint LF_foot_fixed: type fixed, parent LF_FT_wrist, child LF_FOOT, origin xyz=0 0 0 rpy=0 0 0
- added joint LF_ft_joint: type fixed, parent LF_calf, child LF_FT_wrist, origin xyz=0.275 -0.0 -0.278 rpy=0 0 0
- added joint LH_HAA: type revolute, parent base, child LH_hip, origin xyz=-0.301 0.10557 0 rpy=0 0 0, axis 1 0 0, limit lower=-0.7854 upper=0.7854 effort=299 velocity=9.14
- added joint LH_HFE: type revolute, parent LH_hip, child LH_thigh, origin xyz=-0.0795 0.0272 0 rpy=0 0 0, axis 0 1 0, limit lower=-2.618 upper=2.618 effort=299 velocity=9.14
- added joint LH_KFE: type revolute, parent LH_thigh, child LH_calf, origin xyz=-0.24748 0.12015 -0.24752 rpy=0 0 0, axis 0 1 0, limit lower=-1.1345 upper=0.7854 effort=299 velocity=9.14
- added joint LH_foot_fixed: type fixed, parent LH_FT_wrist, child LH_FOOT, origin xyz=0 0 0 rpy=0 0 0
- added joint LH_ft_joint: type fixed, parent LH_calf, child LH_FT_wrist, origin xyz=0.275 -0.0 -0.278 rpy=0 0 0
- added joint RF_HAA: type revolute, parent base, child RF_hip, origin xyz=0.301 -0.10557 0 rpy=0 0 0, axis 1 0 0, limit lower=-0.7854 upper=0.7854 effort=299 velocity=9.14
- added joint RF_HFE: type revolute, parent RF_hip, child RF_thigh, origin xyz=0.0795 -0.0272 0 rpy=0 0 0, axis 0 1 0, limit lower=-2.618 upper=2.618 effort=299 velocity=9.14
- added joint RF_KFE: type revolute, parent RF_thigh, child RF_calf, origin xyz=-0.2475 -0.12015 -0.2475 rpy=0 0 0, axis 0 1 0, limit lower=-1.1345 upper=0.7854 effort=299 velocity=9.14
- added joint RF_foot_fixed: type fixed, parent RF_FT_wrist, child RF_FOOT, origin xyz=0 0 0 rpy=0 0 0
- added joint RF_ft_joint: type fixed, parent RF_calf, child RF_FT_wrist, origin xyz=0.275 -0.0 -0.278 rpy=0 0 0
- added joint RH_HAA: type revolute, parent base, child RH_hip, origin xyz=-0.301 -0.10557 0 rpy=0 0 0, axis 1 0 0, limit lower=-0.7854 upper=0.7854 effort=299 velocity=9.14
- added joint RH_HFE: type revolute, parent RH_hip, child RH_thigh, origin xyz=-0.0795 -0.0272 0 rpy=0 0 0, axis 0 1 0, limit lower=-2.618 upper=2.618 effort=299 velocity=9.14
- added joint RH_KFE: type revolute, parent RH_thigh, child RH_calf, origin xyz=-0.24748 -0.12015 -0.24752 rpy=0 0 0, axis 0 1 0, limit lower=-1.1345 upper=0.7854 effort=299 velocity=9.14
- added joint RH_foot_fixed: type fixed, parent RH_FT_wrist, child RH_FOOT, origin xyz=0 0 0 rpy=0 0 0
- added joint RH_ft_joint: type fixed, parent RH_calf, child RH_FT_wrist, origin xyz=0.275 -0.0 -0.278 rpy=0 0 0
